Commit message: 2 actions implemented, attempt switch to ros humble

File: robot_exploration/urdf/robot5.xacro (robot description, xacro)
@@ -1,8 +1,7 @@
 <?xml version="1.0"?>
-<robot xmlns:xacro="http://www.ros.org/wiki/xacro" name="robot4_xacro">
-<xacro:include filename="$(find robot_exploration)/urdf/robot4.gazebo"/>
+<robot xmlns:xacro="http://www.ros.org/wiki/xacro" name="robot5_xacro">
+<xacro:include filename="$(find robot_exploration)/urdf/robot5.gazebo"/>
 	<xacro:property name="length_wheel" value="0.04" />
 	<xacro:property name="radius_wheel" value="0.1" />
-  <xacro:property name="stick_height" value="0.2" />
 	<xacro:macro name="default_inertial" params="mass">
                <inertial>
@@ -17,4 +16,8 @@
      	</geometry>
 	</xacro:macro>
+  <xacro:macro name="cylinder_inertia" params="mass r l">
+    <inertia ixx="${mass*(3*r*r+l*l)/12}" ixy = "0" ixz = "0"
+                iyy="${mass*(3*r*r+l*l)/12}" iyz = "0" izz="${mass*(r*r)/2}" />
+ </xacro:macro>
   <material name="black">
     <color rgba="0.0 0.0 0.0 1.0"/>
@@ -118,7 +121,7 @@
   <link name="camera_link">
 	    <collision>
-	      <origin xyz="0 0 0.025" rpy="0 0 0"/>
+	      <origin xyz="0 0 0.1" rpy="0 0 0"/>
 	      <geometry>
-		<box size="0.05 0.05 0.05"/>
+		<box size="0.05 0.05 0.2"/>
 	      </geometry>
 	    </collision>
@@ -129,5 +132,5 @@
 	      </geometry>
 	      <material name="red">
-		      <color rgba="1 0 0 1"/>
+		<color rgba="1 0 0 1"/>
 	      </material>
 	    </visual>
@@ -138,61 +141,34 @@
 	    </inertial>
   </link>
-  <link name = "camera_stick">
+  <joint name="camera_joint" type="fixed">
+	    <axis xyz="0 1 0" />
+	    <origin xyz="0.15 0 0.3" rpy="0 0 0"/>
+	    <parent link="link_chassis"/>
+	    <child link="camera_link"/>
+	 </joint>
+  <link name="laser">
+    <inertial>
+      <origin xyz="0 0 0" rpy="0 0 0" />
+      <mass value="1" />
+      <xacro:cylinder_inertia mass="1" r="0.05" l="0.1" />
+    </inertial>
+    <visual>
+      <origin xyz="0 0 0" rpy="0 0 0" />
+      <geometry>
+        <cylinder radius="0.05" length="0.1"/>
+      </geometry>
+      <material name="white" />
+    </visual>
     <collision>
-      <origin xyz = "0 0 0.1" rpy="0 0 0"/>
+      <origin xyz="0 0 0" rpy="0 0 0"/>
       <geometry>
-        <box size = "0.05 0.05 0.1"/>
+        <cylinder radius="0.05" length="0.1"/>
       </geometry>
     </collision>
-    <visual>
-      <origin xyz = "0 0 0.1" rpy="0 0 0"/>
-      <geometry>
-        <box size = "0.05 0.05 0.1"/>
-      </geometry>
-      <material name="orange"/>
-    </visual>
-    <inertial>
-      <mass value="0.05"/>
-      <origin xyz="0 0 0" rpy="0 0 0"/>
-      <inertia ixx="1e-3" ixy="0" ixz="0" iyy="1e-3" iyz="0" izz="1e-3"/>
-    </inertial>
   </link>
-  <joint name="camera_base_joint" type = "fixed">
-    <axis xyz="0 0 1"/>
-    <origin xyz = "0.21 0 0.035" rpy="0 0 0"/>
+  <joint name="joint_laser" type="fixed">
+    <origin xyz="0.15 0 0.2" rpy="0 0 0"/>
     <parent link="link_chassis"/>
-    <child link = "camera_stick"/>
+    <child link="laser"/>
   </joint>
-  <joint name="camera_joint" type="continuous">
-    <axis xyz="0 0 1" />
-    <origin xyz="0 0 0.1" rpy="0 0 0"/>
-    <parent link="camera_stick"/>
-    <child link="camera_link"/>
-  </joint>
-  <!-- <link name = "camera_lens">
-    <collision>
-      <origin xyz="0.005 0 0" rpy="0 0 0"/>
-      <geometry>
-        <box size="0.01 0.025 0.025"/>
-      </geometry>
-    </collision>
-    <visual>
-      <origin xyz="0.005 0 0" rpy="0 0 0"/>
-      <geometry>
-        <box size="0.01 0.025 0.025"/>
-      </geometry>
-      <material name = "black"/>
-    </visual>
-    <inertial>
-      <mass value="1e-7" />
-      <origin xyz="0 0 0" rpy="0 0 0"/>
-      <inertia ixx="1e-8" ixy="0" ixz="0" iyy="1e-8" iyz="0" izz="1e-8" />
-    </inertial>
-  </link>
-  <joint name="camera_lens_joint" type="fixed">
-    <axis xyz="0 0 1" />
-    <origin xyz="0.02 0.0 0.025" rpy="0 0 0"/>
-    <parent link="camera_link"/>
-    <child link="camera_lens"/>
-  </joint> -->
 </robot>
